File: hardware/PSP_Consolizer/consolizer.kicad_pcb (KiCad board)
At the start: 2 copper layers, 52.1 x 37.4 mm, 25 parts, among them J1 right ribbon, J2 Power IN, J3 left ribbon, J4 AVR-ISP-6, J5 Conn_01x06, J6 PS2 Controller, J7 center ribbon, J8 Analog, J9 Power OUT (to PSP), U1 MIC5504-3.3YM5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

Commit message: Modified for PSP 3000 and added Gerber files for JLCPCB
Parts:
- added J10: Conn_01x04, PSP_Consolizer:TE_0-1734839-45_1x04-1MP_P0.5mm_Horizontal, F.Cu at (192.8, 73.9)
- J1: footprint 1-1734592-4:TE_1-1734592-4 -> Connector_FFC-FPC:TE_1-1734839-4_1x14-1MP_P0.5mm_Horizontal
- J3: footprint 1-1734592-0:TE_1-1734592-0 -> PSP_Consolizer:Left_Ribbon
- J7: footprint 1-1734592-0:TE_1-1734592-0 -> Connector_FFC-FPC:TE_1-1734839-0_1x10-1MP_P0.5mm_Horizontal
- S1: footprint L102011ML04Q -> PSP_Consolizer:L102021ML04Q; moved to B.Cu
- U3: footprint MCP4651-103E_ST:SOP65P640X120-14N -> Package_SO:TSSOP-14_4.4x5mm_P0.65mm
- moved S1 7.68 mm to (193.0, 99.8)
- moved J1 1.35 mm to (192.9, 87.3)
- moved J3 1.35 mm to (164.3, 85.9)
- moved J7 1.35 mm to (164.3, 97.0)
Connections:
- J1 pad 1: Net-(J1-Pad1) -> unconnected-(J1-Pad1)
- J1 pad 2: Net-(J1-Pad2) -> unconnected-(J1-Pad2)
- J1 pad 3: Net-(J1-Pad3) -> unconnected-(J1-Pad3)
- J1 pad 4: Net-(J1-Pad4) -> unconnected-(J1-Pad4)
- J1 pad 6: Net-(J1-Pad6) -> unconnected-(J1-Pad6)
- J1 pad 7: Net-(J1-Pad7) -> GND
- J1 pad 8: Net-(J1-Pad8) -> GND
- J5 pad 2: Net-(J5-Pad2) -> unconnected-(J5-Pad2)
- J5 pad 3: Net-(J5-Pad3) -> unconnected-(J5-Pad3)
- J6 pad 1: Net-(J6-Pad1) -> unconnected-(J6-Pad1)
- J6 pad 2: Net-(J6-Pad2) -> unconnected-(J6-Pad2)
- J6 pad 7: Net-(J6-Pad7) -> unconnected-(J6-Pad7)
- S1 pad 1: Net-(S1-Pad1) -> unconnected-(S1-Pad1)
- U1 pad 4: Net-(U1-Pad4) -> unconnected-(U1-Pad4)
- U2 pad 20: Net-(U2-Pad20) -> unconnected-(U2-Pad20)
- U3 pad 11: Net-(U3-Pad11) -> unconnected-(U3-Pad11)
Routing:
- net Net-(J3-Pad2): track 28.3 -> 21.9 mm, vias 2 -> 1
- net Net-(J8-Pad1): track 6.12 -> 11.0 mm
- net Net-(J8-Pad3): track 6.17 -> 9.52 mm
- net Net-(J8-Pad2): track 10.7 -> 13.5 mm
Other:
- board size 52.1 x 37.4 mm -> 52 x 37.2 mm
- net class Default removed
- board text added: "Analog"
- board text added: "JLCJLCJLCJLC"
